File: pcb/keyboard.kicad_pcb (KiCad board)
At the start: 2 copper layers, 150.5 x 136.3 mm, 68 parts, among them SW1 SW_Push

Commit message: Added traces for rows (kinda important ;_;)
Connections:
- ProMicroBottom1 pad 14: Net-(ProMicroBottom1-Pad14) -> row0
- ProMicroBottom1 pad 15: Net-(ProMicroBottom1-Pad15) -> row1
- ProMicroBottom1 pad 16: Net-(ProMicroBottom1-Pad16) -> row2
- ProMicroBottom1 pad 17: Net-(ProMicroBottom1-Pad17) -> row3
- ProMicroBottom1 pad 18: Net-(ProMicroBottom1-Pad18) -> row4
- ProMicroTop1 pad 14: Net-(ProMicroTop1-Pad14) -> row0
- ProMicroTop1 pad 15: Net-(ProMicroTop1-Pad15) -> row1
- ProMicroTop1 pad 16: Net-(ProMicroTop1-Pad16) -> row2
- ProMicroTop1 pad 17: Net-(ProMicroTop1-Pad17) -> row3
- ProMicroTop1 pad 18: Net-(ProMicroTop1-Pad18) -> row4
Routing:
- net row4: track 138.4 -> 250.4 mm
- net row3: track 110.4 -> 213.5 mm
- net row2: track 110.4 -> 191.1 mm
- net row1: track 110.4 -> 169.1 mm
- net row0: track 110.4 -> 152.2 mm
- net RST: track 48.3 -> 49.7 mm
